File: pcb.kicad_sch (KiCad schematic)
At the start: 3 parts

Commit message: inital layout
Parts:
- removed BT1: CR2032, Battery:BatteryHolder_Keystone_3034_1x20mm, symbol Device:Battery_Cell
- removed D1: LED, LED_SMD:LED_0805_2012Metric, symbol Device:LED
- removed R1: 1k, Resistor_SMD:R_0805_2012Metric, symbol Device:R
- added C10, C21, C22, C9: 100n, Capacitor_SMD:C_0402_1005Metric, symbol Device:C_Small
- added C11: 4u7, Capacitor_SMD:C_0402_1005Metric, symbol Device:C_Small
- added C19: 1u, Capacitor_SMD:C_0402_1005Metric, symbol Device:C_Small
- added C20, C8: 10u tantalum, Capacitor_Tantalum_SMD:CP_EIA-3216-10_Kemet-I, symbol Device:C_Polarized_Small
- added C7: 10u, Capacitor_SMD:C_0402_1005Metric, symbol Device:C_Small
- added FB1: 100R@100MHz, Resistor_SMD:R_0805_2012Metric, symbol Device:FerriteBead_Small
- added H1, H2, H3: MountingHole, MountingHole:MountingHole_2.2mm_M2, symbol Mechanical:MountingHole
- added J2: USB_C_Receptacle_USB2.0, Connector_USB:USB_C_Receptacle_HRO_TYPE-C-31-M-12, symbol Connector:USB_C_Receptacle_USB2.0
- added R1, R2: 5k1, Resistor_SMD:R_0402_1005Metric, symbol Device:R_Small
- added R10, R11: 4k7, Capacitor_SMD:C_0402_1005Metric, symbol Device:R_Small
- added R12, R5: 10k, Capacitor_SMD:C_0402_1005Metric, symbol Device:R_Small
- added R15, R16, R17, R18: 100k, Capacitor_SMD:C_0402_1005Metric, symbol Device:R_Small
- added SW1: SW_Push, Button_Switch_SMD:SW_Push_1P1T_NO_CK_KSC7xxJ, symbol Switch:SW_Push
- added TP1: Batt+, TestPoint:TestPoint_THTPad_2.0x2.0mm_Drill1.0mm, symbol Connector:TestPoint
- added TP2: Batt-, TestPoint:TestPoint_THTPad_2.0x2.0mm_Drill1.0mm, symbol Connector:TestPoint
- added U1: ADXL375, Package_LGA:LGA-14_3x5mm_P0.8mm_LayoutBorder1x6y, symbol Sensor_Motion:ADXL343
- added U2: ESP32-S3-MINI-1, PCM_Espressif:ESP32-S2-MINI-1, symbol PCM_Espressif:ESP32-S3-MINI-1
- added U3: AMS1117-3.3, Package_TO_SOT_SMD:SOT-223-3_TabPin2, symbol Regulator_Linear:AMS1117-3.3
- added U4: MCP73831-2-OT, Package_TO_SOT_SMD:SOT-23-5, symbol Battery_Management:MCP73831-2-OT
- added U5: W25Q128JVS, Package_SO:SOIC-8_5.23x5.23mm_P1.27mm, symbol Memory_Flash:W25Q128JVS
Connections:
- net GND: now also C10.2, C11.2, C19.2, C20.2, C21.2, C22.2, C7.2, C8.2, C9.2, J2.A1 (GND), J2.A12 (GND), J2.B1 (GND), J2.B12 (GND), R1.2, R16.2, R18.2, R2.1, R5.2, SW1.1, TP2.1, U1.11 (RES), U1.2 (GND), U1.4 (GND), U1.5 (GND), U2.1 (GND), U2.2 (GND), U2.42 (GND), U2.43 (GND), U2.46 (GND), U2.47 (GND), U2.48 (GND), U2.49 (GND), U2.50 (GND), U2.51 (GND), U2.52 (GND), U2.53 (GND), U2.54 (GND), U2.55 (GND), U2.56 (GND), U2.57 (GND), U2.58 (GND), U2.59 (GND), U2.60 (GND), U2.61 (GND), U2.62 (GND), U2.63 (GND), U2.64 (GND), U2.65 (GND), U3.1 (GND), U4.2 (V_{SS}), U5.4 (GND)
- new net: C19.1, R12.2, U2.45 (EN)
- new net: J2.B5 (CC2), R2.2
- new net: R5.1, U4.5 (PROG)
- new net: FB1.1, J2.A4 (VBUS), J2.A9 (VBUS), J2.B4 (VBUS), J2.B9 (VBUS)
- new net: J2.A5 (CC1), R1.1
- new net +3.3V: C10.1, C20.1, C21.1, C22.1, C8.1, R10.1, R11.1, R12.1, U1.1 (Vdd_I/O), U1.3 (RES), U1.6 (Vs), U2.3 (3V3), U3.2 (VO), U5.8 (VCC)
- new net ACCEL-INT1: U1.8 (INT1), U2.13 (GPIO9/TOUCH9/ADC1_CH8/FSPIHD/SUBSPIHD)
- new net ACCEL-INT2: U1.9 (INT2), U2.12 (GPIO8/TOUCH8/ADC1_CH7/SUBSPICS1)
- new net ACCEL-SCK: U1.14 (SCL/SCLK), U2.9 (GPIO5/TOUCH5/ADC1_CH4)
- new net ACCEL-SDI: U1.13 (SDA/SDI/SDIO), U2.10 (GPIO6/TOUCH6/ADC1_CH5)
- new net ACCEL-SDO: U1.12 (SDO/ADDR), U2.11 (GPIO7/TOUCH7/ADC1_CH6)
- new net ACCEL-nCS: U1.7 (~{CS}), U2.14 (GPIO10/TOUCH10/ADC1_CH9/FSPICS0/FSPIIO4/SUBSPICS0)
- new net BOOT: SW1.2, U2.4 (GPIO0/BOOT)
- new net CHARGE_STAT: U2.17 (GPIO13/TOUCH13/ADC2_CH2/FSPIQ/FSPIIO7/SUBSPIQ), U4.1 (STAT)
- new net FLASH-SCK: U2.39 (U0TXD/GPIO43/CLK_OUT1), U5.6 (CLK)
- new net FLASH-SDI: U2.38 (MTMS/GPIO42), U5.5 (DI(IO0))
- new net FLASH-SDO: U2.40 (U0RXD/GPIO44/CLK_OUT2), U5.2 (DO(IO1))
- new net FLASH-nCS: U2.41 (GPIO45), U5.1 (~{CS})
- new net I2C_SCL: R11.2, U2.31 (SPIIO6/GPIO35/FSPID/SUBSPID)
- new net I2C_SDA: R10.2, U2.29 (SPIIO5/GPIO34/FSPICS0/SUBSPICS0)
- new net LED_D: U2.5 (GPIO1/TOUCH1/ADC1_CH0)
- new net LED_EN: U2.35 (MTCK/GPIO39/CLK_OUT3/SUBSPICS1)
- new net OLED_ENABLE: U2.26 (GPIO26)
- new net OLED_RESET: U2.27 (GPIO47/SPICLK_P/SUBSPICLK_P_DIFF)
- new net USB_D+: J2.A6 (D+), J2.B6 (D+), U2.24 (GPIO20/U1CTS/ADC2_CH9/CLK_OUT1/USB_D+)
- new net USB_D-: J2.A7 (D-), J2.B7 (D-), U2.23 (GPIO19/U1RTS/ADC2_CH8/CLK_OUT2/USB_D-)
- new net USB_VBUS: C11.1, FB1.2, R17.1, U4.4 (V_{DD})
- new net VBAT: C7.1, C9.1, R15.1, TP1.1, U3.3 (VI), U4.3 (V_{BAT})
- new net VBAT_MEAS: R15.2, R16.1, U2.7 (GPIO3/TOUCH3/ADC1_CH2)
- new net VBUS_MEAS: R17.2, R18.1, U2.8 (GPIO4/TOUCH4/ADC1_CH3)
- no-connect marks 0 -> 22
Other:
- added sheet LEDs (leds.kicad_sch)
- added sheet OLED (OLED.kicad_sch)
- note added: "3V3 LDO"
- note added: "Accelerometer"
- note added: "Battery & USB Voltage measurement"
- note added: "Battery connection"
- note added: "Extra external SPI flash"
- note added: "OLED Display"
- note added: "RC network to delay startup"
- note added: "USB Type-C and battery charger"
- note added: "Use 16V or higher tantalum capacitors"
- note added: "WS2812 LEDs"
