File: pcb.kicad_sch (KiCad schematic)
At the start: 32 parts, among them J2 USB_C_Receptacle_USB2.0, SW1 SW_Push, U1 ADXL375, U2 ESP32-S3-MINI-1, U3 AMS1117-3.3, U4 MCP73831-2-OT, U5 W25Q128JVS

Commit message: fixed library issues
Parts:
- U2: footprint PCM_Espressif:ESP32-S2-MINI-1 -> Espressif:ESP32-S3-MINI-1; symbol PCM_Espressif:ESP32-S3-MINI-1 -> Espressif:ESP32-S3-MINI-1
Changed lines of the file:
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@@
     )
   )
-  (symbol (lib_id "PCM_Espressif:ESP32-S3-MINI-1") (at 114.3 173.99 0) (unit 1)
+  (symbol (lib_id "Espressif:ESP32-S3-MINI-1") (at 114.3 173.99 0) (unit 1)
     (in_bom yes) (on_board yes) (dnp no) (fields_autoplaced)
     (property "Reference" "U2" (at 116.2559 130.81 0)
@@
       (effects (font (size 1.27 1.27)) (justify left))
     )
-    (property "Footprint" "PCM_Espressif:ESP32-S2-MINI-1" (at 114.3 229.87 0)
+    (property "Footprint" "Espressif:ESP32-S3-MINI-1" (at 114.3 229.87 0)
       (effects (font (size 1.27 1.27)) hide)
     )

Commit message: added part numbers
Parts:
- C10, C21, C22, C9: LCSC (none) -> C1525
- C11: LCSC (none) -> C23733
- C19: LCSC (none) -> C52923
- C20, C8: LCSC (none) -> C7171
- C7: LCSC (none) -> C15525
- R10, R11: value 4k7 -> 10k; footprint Capacitor_SMD:C_0402_1005Metric -> Resistor_SMD:R_0402_1005Metric; LCSC (none) -> C25086
- R12, R5: footprint Capacitor_SMD:C_0402_1005Metric -> Resistor_SMD:R_0402_1005Metric; LCSC (none) -> C25086
- R15, R16, R17, R18: value 100k -> 120k; footprint Capacitor_SMD:C_0402_1005Metric -> Resistor_SMD:R_0402_1005Metric; LCSC (none) -> C25750
- U1: LCSC (none) -> C481898
- U2: LCSC (none) -> C3013941
- U3: LCSC (none) -> C6186
- U4: LCSC (none) -> C841234
Changed lines of the file:
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@@
+      (effects (font (size 1.27 1.27)) hide)
+    )
+    (property "LCSC" "C6186" (at 255.27 45.72 0)
       (effects (font (size 1.27 1.27)) hide)
     )
@@
       (effects (font (size 1.27 1.27)) (justify left))
     )
-    (property "Footprint" "Capacitor_SMD:C_0402_1005Metric" (at 53.34 133.35 0)
+    (property "Footprint" "Resistor_SMD:R_0402_1005Metric" (at 53.34 133.35 0)
       (effects (font (size 1.27 1.27)) hide)
     )
     (property "Datasheet" "~" (at 53.34 133.35 0)
+      (effects (font (size 1.27 1.27)) hide)
+    )
+    (property "LCSC" "C25086" (at 53.34 133.35 0)
       (effects (font (size 1.27 1.27)) hide)
     )
@@
     )
     (property "Datasheet" "~" (at 123.19 50.8 0)
+      (effects (font (size 1.27 1.27)) hide)
+    )
+    (property "LCSC" "C23733" (at 123.19 50.8 0)
       (effects (font (size 1.27 1.27)) hide)
     )
@@
       (effects (font (size 1.27 1.27)) (justify right))
     )
-    (property "Value" "100k" (at 229.87 78.74 0)
+    (property "Value" "120k" (at 229.87 78.74 0)
       (effects (font (size 1.27 1.27)) (justify right))
     )
-    (property "Footprint" "Capacitor_SMD:C_0402_1005Metric" (at 227.33 77.47 0)
+    (property "Footprint" "Resistor_SMD:R_0402_1005Metric" (at 227.33 77.47 0)
       (effects (font (size 1.27 1.27)) hide)
     )
     (property "Datasheet" "~" (at 227.33 77.47 0)
+      (effects (font (size 1.27 1.27)) hide)
+    )
+    (property "LCSC" "C25750" (at 227.33 77.47 0)
       (effects (font (size 1.27 1.27)) hide)
     )
@@
       (effects (font (size 1.27 1.27)) (justify left))
     )
-    (property "Footprint" "Capacitor_SMD:C_0402_1005Metric" (at 125.73 60.96 0)
+    (property "Footprint" "Resistor_SMD:R_0402_1005Metric" (at 125.73 60.96 0)
       (effects (font (size 1.27 1.27)) hide)
     )
     (property "Datasheet" "~" (at 125.73 60.96 0)
+      (effects (font (size 1.27 1.27)) hide)
+    )
+    (property "LCSC" "C25086" (at 125.73 60.96 0)
       (effects (font (size 1.27 1.27)) hide)
     )
@@
       (effects (font (size 1.27 1.27)) hide)
     )
+    (property "LCSC" "C15525" (at 231.14 49.53 0)
+      (effects (font (size 1.27 1.27)) hide)
+    )
     (pin "1")
     (pin "2")
@@
       (effects (font (size 1.27 1.27)) (justify left))
     )
-    (property "Value" "4k7" (at 224.79 125.73 0)
-      (effects (font (size 1.27 1.27)) (justify left))
-    )
-    (property "Footprint" "Capacitor_SMD:C_0402_1005Metric" (at 222.25 124.46 0)
+    (property "Value" "10k" (at 224.79 125.73 0)
+      (effects (font (size 1.27 1.27)) (justify left))
+    )
+    (property "Footprint" "Resistor_SMD:R_0402_1005Metric" (at 222.25 124.46 0)
       (effects (font (size 1.27 1.27)) hide)
     )
     (property "Datasheet" "~" (at 222.25 124.46 0)
+      (effects (font (size 1.27 1.27)) hide)
+    )
+    (property "LCSC" "C25086" (at 222.25 124.46 0)
       (effects (font (size 1.27 1.27)) hide)
     )
@@
     )
     (property "Datasheet" "~" (at 53.34 143.51 0)
+      (effects (font (size 1.27 1.27)) hide)
+    )
+    (property "LCSC" "C52923" (at 53.34 143.51 0)
       (effects (font (size 1.27 1.27)) hide)
     )
@@
       (effects (font (size 1.27 1.27)) (justify right))
     )
-    (property "Value" "100k" (at 229.87 88.9 0)
+    (property "Value" "120k" (at 229.87 88.9 0)
       (effects (font (size 1.27 1.27)) (justify right))
     )
-    (property "Footprint" "Capacitor_SMD:C_0402_1005Metric" (at 227.33 87.63 0)
+    (property "Footprint" "Resistor_SMD:R_0402_1005Metric" (at 227.33 87.63 0)
       (effects (font (size 1.27 1.27)) hide)
     )
     (property "Datasheet" "~" (at 227.33 87.63 0)
+      (effects (font (size 1.27 1.27)) hide)
+    )
+    (property "LCSC" "C25750" (at 227.33 87.63 0)
       (effects (font (size 1.27 1.27)) hide)
     )
@@
       (effects (font (size 1.27 1.27)) (justify right))
     )
-    (property "Value" "100k" (at 252.73 78.74 0)
+    (property "Value" "120k" (at 252.73 78.74 0)
       (effects (font (size 1.27 1.27)) (justify right))
     )
-    (property "Footprint" "Capacitor_SMD:C_0402_1005Metric" (at 250.19 77.47 0)
+    (property "Footprint" "Resistor_SMD:R_0402_1005Metric" (at 250.19 77.47 0)
       (effects (font (size 1.27 1.27)) hide)
     )
     (property "Datasheet" "~" (at 250.19 77.47 0)
+      (effects (font (size 1.27 1.27)) hide)
+    )
+    (property "LCSC" "C25750" (at 250.19 77.47 0)
       (effects (font (size 1.27 1.27)) hide)
     )
@@
     )
     (property "Datasheet" "~" (at 265.43 49.53 0)
+      (effects (font (size 1.27 1.27)) hide)
+    )
+    (property "LCSC" "C7171" (at 265.43 49.53 0)
       (effects (font (size 1.27 1.27)) hide)
     )
@@
       (effects (font (size 1.27 1.27)) hide)
     )
+    (property "LCSC" "C841234" (at 142.24 55.88 0)
+      (effects (font (size 1.27 1.27)) hide)
+    )
     (pin "1")
     (pin "2")
@@
       (effects (font (size 1.27 1.27)) hide)
     )
+    (property "LCSC" "C1525" (at 97.79 125.73 0)
+      (effects (font (size 1.27 1.27)) hide)
+    )
     (pin "1")
     (pin "2")
@@
     )
     (property "Datasheet" "https://www.analog.com/media/en/technical-documentation/data-sheets/ADXL343.pdf" (at 238.76 200.66 0)
+      (effects (font (size 1.27 1.27)) hide)
+    )
+    (property "LCSC" "C481898" (at 238.76 200.66 0)
       (effects (font (size 1.27 1.27)) hide)
     )
@@
       (effects (font (size 1.27 1.27)) hide)
     )
+    (property "LCSC" "C1525" (at 241.3 49.53 0)
+      (effects (font (size 1.27 1.27)) hide)
+    )
     (pin "1")
     (pin "2")
@@
       (effects (font (size 1.27 1.27)) hide)
     )
+    (property "LCSC" "C1525" (at 273.05 200.66 0)
+      (effects (font (size 1.27 1.27)) hide)
+    )
     (pin "1")
     (pin "2")
@@
     )
     (property "Datasheet" "https://www.espressif.com/sites/default/files/documentation/esp32-s3-mini-1_mini-1u_datasheet_en.pdf" (at 114.3 232.41 0)
+      (effects (font (size 1.27 1.27)) hide)
+    )
+    (property "LCSC" "C3013941" (at 114.3 173.99 0)
       (effects (font (size 1.27 1.27)) hide)
     )
@@
       (effects (font (size 1.27 1.27)) (justify left))
     )
-    (property "Value" "4k7" (at 233.68 125.73 0)
-      (effects (font (size 1.27 1.27)) (justify left))
-    )
-    (property "Footprint" "Capacitor_SMD:C_0402_1005Metric" (at 231.14 124.46 0)
+    (property "Value" "10k" (at 233.68 125.73 0)
+      (effects (font (size 1.27 1.27)) (justify left))
+    )
+    (property "Footprint" "Resistor_SMD:R_0402_1005Metric" (at 231.14 124.46 0)
       (effects (font (size 1.27 1.27)) hide)
     )
@@
       (effects (font (size 1.27 1.27)) hide)
     )
+    (property "LCSC" "C25086" (at 231.14 124.46 0)
+      (effects (font (size 1.27 1.27)) hide)
+    )
     (pin "1")
     (pin "2")
@@
     )
     (property "Datasheet" "~" (at 283.21 49.53 0)
+      (effects (font (size 1.27 1.27)) hide)
+    )
+    (property "LCSC" "C7171" (at 283.21 49.53 0)
       (effects (font (size 1.27 1.27)) hide)
     )
@@
     )
     (property "Datasheet" "~" (at 260.35 245.11 0)
+      (effects (font (size 1.27 1.27)) hide)
+    )
+    (property "LCSC" "C1525" (at 260.35 245.11 0)
       (effects (font (size 1.27 1.27)) hide)
     )
@@
       (effects (font (size 1.27 1.27)) (justify right))
     )
-    (property "Value" "100k" (at 252.73 88.9 0)
+    (property "Value" "120k" (at 252.73 88.9 0)
       (effects (font (size 1.27 1.27)) (justify right))
     )
-    (property "Footprint" "Capacitor_SMD:C_0402_1005Metric" (at 250.19 87.63 0)
+    (property "Footprint" "Resistor_SMD:R_0402_1005Metric" (at 250.19 87.63 0)
       (effects (font (size 1.27 1.27)) hide)
     )
@@
       (effects (font (size 1.27 1.27)) hide)
     )
+    (property "LCSC" "C25750" (at 250.19 87.63 0)
+      (effects (font (size 1.27 1.27)) hide)
+    )

Commit message: Bare ESP layout
Parts:
- removed C19: 1u, Capacitor_SMD:C_0402_1005Metric, symbol Device:C_Small
- removed C21: 100n, Capacitor_SMD:C_0402_1005Metric, symbol Device:C_Small
- removed R12: 10k, Resistor_SMD:R_0402_1005Metric, symbol Device:R_Small
- removed U2: ESP32-S3-MINI-1, Espressif:ESP32-S3-MINI-1, symbol Espressif:ESP32-S3-MINI-1
- added AE2: PCB Antenna, RF_Antenna:Texas_SWRA117D_2.4GHz_Left, symbol Device:Antenna_Loop
- added C23, C24, C26, C29, C32, C38, C39: 100n, Capacitor_SMD:C_0402_1005Metric, symbol Device:C_Small
- added C25, C27, C31, C33: 1u, Capacitor_SMD:C_0402_1005Metric, symbol Device:C_Small
- added C28, C30: 10u, Capacitor_SMD:C_0402_1005Metric, symbol Device:C_Small
- added C34, C35: 22p, Capacitor_SMD:C_0402_1005Metric, symbol Device:C_Small
- added C36: 4p7, Capacitor_SMD:C_0402_1005Metric, symbol Device:C_Small
- added C37: 3p3, Capacitor_SMD:C_0402_1005Metric, symbol Device:C_Small
- added H4: MountingHole, MountingHole:MountingHole_2.2mm_M2, symbol Mechanical:MountingHole
- added L1, L2: 3.9nH, Inductor_SMD:L_0402_1005Metric, symbol Device:L_Small
- added L3: 15nH, Inductor_SMD:L_0402_1005Metric, symbol Device:L_Small
- added L4: 1.8nH, Inductor_SMD:L_0402_1005Metric, symbol Device:L_Small
- added R13, R14: 10k, Resistor_SMD:R_0402_1005Metric, symbol Device:R_Small
- added R20: 470, Resistor_SMD:R_0402_1005Metric, symbol Device:R_Small
- added R21, R22: 0R, Resistor_SMD:R_0402_1005Metric, symbol Device:R_Small
- added TP3: TXD, TestPoint:TestPoint_Pad_D1.0mm, symbol Connector:TestPoint
- added TP4: RXD, TestPoint:TestPoint_Pad_D1.0mm, symbol Connector:TestPoint
- added TP5: BOOT1, TestPoint:TestPoint_Pad_D1.0mm, symbol Connector:TestPoint
- added U6: ESP32-S3, Package_DFN_QFN:QFN-56-1EP_7x7mm_P0.4mm_EP5.6x5.6mm, symbol Espressif:ESP32-S3
- added Y1: 40MHz 15pF, Crystal:Crystal_SMD_3225-4Pin_3.2x2.5mm, symbol Device:Crystal_GND24
- C22, U5: now fitted
Connections:
- net +3.3V: now also C23.1, C26.1, C27.1, C28.1, C30.1, C31.1, C32.1, L1.1, L2.1, R14.1, U6.20 (VDD3P3_RTC), U6.46 (VDD3P3_CPU), U6.55 (VDDA), U6.56 (VDDA)
- net ACCEL-INT1: now also U6.41 (GPIO36)
- net ACCEL-INT2: now also U6.40 (GPIO35)
- net ACCEL-SCK: now also U6.37 (SPICLK_P/GPIO47)
- net ACCEL-SDI: now also U6.38 (GPIO33)
- net ACCEL-SDO: now also U6.39 (GPIO34)
- net ACCEL-nCS: now also U6.42 (GPIO37)
- net BOOT: now also U6.5 (GPIO0/BOOT)
- net CHARGE_STAT: now also U6.17 (GPIO12/ADC2_CH1)
- net FLASH-nCS: now also U6.32 (SPICS0/GPIO29)
- net GND: now also AE2.2, C23.2, C24.2, C25.2, C26.2, C27.2, C28.2, C29.2, C30.2, C31.2, C32.2, C33.2, C34.1, C35.2, C36.2, C37.2, C38.2, C39.2, R13.2, U6.57 (GND), Y1.2, Y1.4
- net I2C_SCL: now also U6.44 (MTCK/JTAG/GPIO39)
- net I2C_SDA: now also U6.43 (GPIO38)
- net OLED_ENABLE: now also U6.19 (GPIO14/ADC2_CH3)
- net OLED_RESET: now also U6.45 (MTDO/JTAG/GPIO40)
- net USB_D+: now also R21.2
- net USB_D-: now also R22.2
- net VBAT_MEAS: now also C39.1, U6.9 (GPIO4/ADC1_CH3)
- net VBUS_MEAS: now also C38.1, U6.10 (GPIO5/ADC1_CH4)
- net FLASH-WP: now reaches U5.3 (IO2)
- net FLASH-WP: now also U6.31 (SPIWP/GPIO28)
- net FLASH-HD: now reaches U5.7 (IO3)
- net FLASH-HD: now also U6.30 (SPIHD/GPIO27)
- net FLASH-SCK renamed FLASH-CLK
- net FLASH-CLK: now also U6.33 (SPICLK/GPIO30)
- net FLASH-SDI renamed FLASH-D
- net FLASH-D: now also U6.35 (SPID/GPIO32)
- net FLASH-SDO renamed FLASH-Q
- net FLASH-Q: now also U6.34 (SPIQ/GPIO31)
- new net: C34.2, L3.1, Y1.3
- new net: L3.2, U6.54 (XTAL_P)
- new net: R20.1, U6.49 (U0TXD/PROG/GPIO43)
- new net: R20.2, TP3.1
- new net: C33.1, R14.2, U6.4 (CHIP_PU/RESET)
- new net: R22.1, U6.25 (GPIO19/USB_D-/ADC2_CH8)
- new net: R21.1, U6.26 (GPIO20/USB_D+/ADC2_CH9)
- new net: TP4.1, U6.50 (U0RXD/PROG/GPIO44)
- new net: R13.1, U6.51 (GPIO45)
- new net: C35.1, U6.53 (XTAL_N), Y1.1
- new net: TP5.1, U6.52 (GPIO46)
- new net ANT_RF: AE2.1, C37.1, L4.1
- new net ESP_RF: C36.1, L4.2, U6.1 (LNA_IN/RF)
- new net VDD3P3: C29.1, L1.2, L2.2, U6.2 (VDD3P3), U6.3 (VDD3P3)
- new net VDD_SPI: C24.1, C25.1, U6.29 (VDD_SPI)
- no-connect marks 22 -> 21
Other:
- removed sheet LEDs
- note added: "Pi matching network Q=2.6 Source impedance=30+10J"
- note added: "SPI Flash"
- note added: "Sets SPI Flash voltage to 3.3V"
- note removed: "Extra external SPI flash"
- note removed: "WS2812 LEDs"
- moved on the sheet: SW1

Commit message: fix erc/drc
Connections:
- no-connect marks 21 -> 22
Changed lines of the file:
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@@
   (no_connect (at 92.71 177.8))
   (no_connect (at 158.75 218.44))
+  (no_connect (at 158.75 213.36))
   (no_connect (at 158.75 200.66))
   (no_connect (at 158.75 208.28))

Commit message: added part numbers
Parts:
- L2: LCSC (none) -> C14033
- L3: LCSC (none) -> C27143
- R20: LCSC (none) -> C25117
- R21, R22: LCSC (none) -> C17168
- U5: LCSC (none) -> C97521
- U6: LCSC (none) -> C2913192
Changed lines of the file:
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@@
       (effects (font (size 1.27 1.27)) hide)
     )
-    (property "LCSC" "" (at 87.63 187.96 90)
+    (property "LCSC" "C27143" (at 87.63 187.96 90)
       (effects (font (size 1.27 1.27)) hide)
     )
@@
       (effects (font (size 1.27 1.27)) hide)
     )
+    (property "LCSC" "C25117" (at 167.64 165.1 0)
+      (effects (font (size 1.27 1.27)) hide)
+    )
     (pin "1")
     (pin "2")
@@
     )
     (property "Datasheet" "http://www.winbond.com/resource-files/w25q128jv_dtr%20revc%2003272018%20plus.pdf" (at 234.95 245.11 0)
+      (effects (font (size 1.27 1.27)) hide)
+    )
+    (property "LCSC" "C97521" (at 234.95 245.11 0)
       (effects (font (size 1.27 1.27)) hide)
     )
@@
       (effects (font (size 1.27 1.27)) hide)
     )
+    (property "LCSC" "C17168" (at 166.37 175.26 0)
+      (effects (font (size 1.27 1.27)) hide)
+    )
     (pin "1")
     (pin "2")
@@
     )
     (property "Datasheet" "~" (at 166.37 172.72 0)
+      (effects (font (size 1.27 1.27)) hide)
+    )
+    (property "LCSC" "C17168" (at 166.37 172.72 0)
       (effects (font (size 1.27 1.27)) hide)
     )
@@
     )
     (property "Datasheet" "https://www.espressif.com/sites/default/files/documentation/esp32-s3_datasheet_en.pdf" (at 125.73 251.46 0)
+      (effects (font (size 1.27 1.27)) hide)
+    )
+    (property "LCSC" "C2913192" (at 125.73 200.66 0)
       (effects (font (size 1.27 1.27)) hide)
     )
@@
       (effects (font (size 1.27 1.27)) hide)
     )
+    (property "LCSC" "C14033" (at 105.41 133.35 0)
+      (effects (font (size 1.27 1.27)) hide)
+    )
