File: OLED.kicad_sch (KiCad schematic)
At the start: 13 parts, among them J2 OLED, Q3 2N7002, Q4 Si2301CDS

Commit message: Use bare ESP32 chip instead of module (#1)
* fixed library issues

* add submodules to CI/CD

* fix yaml syntax

* added part numbers

* Bare ESP layout

* fix erc/drc

* fix overlap

* added part numbers

* fixed layout
Parts:
- C12, C17: LCSC (none) -> C23733
- C13, C18: LCSC (none) -> C1525
- C14: LCSC (none) -> C12530
- C15, C16: LCSC (none) -> C52923
- Q3: LCSC (none) -> C8545
- Q4: LCSC (none) -> C10487
- R3, R8: footprint Capacitor_SMD:C_0402_1005Metric -> Resistor_SMD:R_0402_1005Metric; LCSC (none) -> C25086
- R9: footprint Capacitor_SMD:C_0402_1005Metric -> Resistor_SMD:R_0402_1005Metric; LCSC (none) -> C912013
Changed lines of the file:
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@@
           (reference "#PWR021") (unit 1)
         )
-        (path "/74bf6178-dca6-4427-901b-44badacb7eee/2156e343-9b45-4780-9034-2535dd910fa6"
-          (reference "#PWR020") (unit 1)
-        )
         (path "/74bf6178-dca6-4427-901b-44badacb7eee/7d25a774-c98a-421e-98be-59f63435153d"
           (reference "#PWR021") (unit 1)
@@
       (effects (font (size 1.27 1.27)) hide)
     )
+    (property "LCSC" "C52923" (at 153.67 62.23 0)
+      (effects (font (size 1.27 1.27)) hide)
+    )
     (pin "1")
     (pin "2")
@@
     )
     (property "Datasheet" "~" (at 165.1 57.15 0)
+      (effects (font (size 1.27 1.27)) hide)
+    )
+    (property "LCSC" "C52923" (at 165.1 57.15 0)
       (effects (font (size 1.27 1.27)) hide)
     )
@@
     )
     (property "Datasheet" "~" (at 154.94 95.25 0)
+      (effects (font (size 1.27 1.27)) hide)
+    )
+    (property "LCSC" "C12530" (at 154.94 95.25 0)
       (effects (font (size 1.27 1.27)) hide)
     )
@@
       (effects (font (size 1.27 1.27)) (justify right))
     )
-    (property "Footprint" "Capacitor_SMD:C_0402_1005Metric" (at 124.46 55.88 0)
+    (property "Footprint" "Resistor_SMD:R_0402_1005Metric" (at 124.46 55.88 0)
       (effects (font (size 1.27 1.27)) hide)
     )
@@
       (effects (font (size 1.27 1.27)) hide)
     )
+    (property "LCSC" "C25086" (at 124.46 55.88 0)
+      (effects (font (size 1.27 1.27)) hide)
+    )
     (pin "1")
     (pin "2")
@@
           (reference "R8") (unit 1)
         )
-        (path "/74bf6178-dca6-4427-901b-44badacb7eee/2156e343-9b45-4780-9034-2535dd910fa6"
-          (reference "R2") (unit 1)
-        )
         (path "/74bf6178-dca6-4427-901b-44badacb7eee/7d25a774-c98a-421e-98be-59f63435153d"
           (reference "R8") (unit 1)
@@
         (path "/74bf6178-dca6-4427-901b-44badacb7eee"
           (reference "#PWR023") (unit 1)
-        )
-        (path "/74bf6178-dca6-4427-901b-44badacb7eee/2156e343-9b45-4780-9034-2535dd910fa6"
-          (reference "#PWR05") (unit 1)
         )
         (path "/74bf6178-dca6-4427-901b-44badacb7eee/7d25a774-c98a-421e-98be-59f63435153d"
@@
       (effects (font (size 1.27 1.27)) hide)
     )
+    (property "LCSC" "C23733" (at 115.57 90.17 0)
+      (effects (font (size 1.27 1.27)) hide)
+    )
     (pin "1")
     (pin "2")
@@
       (effects (font (size 1.27 1.27)) (justify left))
     )
-    (property "Footprint" "Capacitor_SMD:C_0402_1005Metric" (at 140.97 95.25 0)
+    (property "Footprint" "Resistor_SMD:R_0402_1005Metric" (at 140.97 95.25 0)
       (effects (font (size 1.27 1.27)) hide)
     )
     (property "Datasheet" "~" (at 140.97 95.25 0)
+      (effects (font (size 1.27 1.27)) hide)
+    )
+    (property "LCSC" "C912013" (at 140.97 95.25 0)
       (effects (font (size 1.27 1.27)) hide)
     )
@@
       (effects (font (size 1.27 1.27)) hide)
     )
+    (property "LCSC" "C1525" (at 172.72 95.25 0)
+      (effects (font (size 1.27 1.27)) hide)
+    )
     (pin "1")
     (pin "2")
@@
       (effects (font (size 1.27 1.27)) hide)
     )
+    (property "LCSC" "C23733" (at 163.83 95.25 0)
+      (effects (font (size 1.27 1.27)) hide)
+    )
     (pin "1")
     (pin "2")
@@
     )
     (property "Datasheet" "~" (at 124.46 90.17 0)
+      (effects (font (size 1.27 1.27)) hide)
+    )
+    (property "LCSC" "C1525" (at 124.46 90.17 0)
       (effects (font (size 1.27 1.27)) hide)
     )
@@
       (effects (font (size 1.27 1.27)) (justify left) hide)
     )
+    (property "LCSC" "C8545" (at 121.92 71.12 0)
+      (effects (font (size 1.27 1.27)) hide)
+    )
     (pin "1")
     (pin "2")
@@
           (reference "Q3") (unit 1)
         )
-        (path "/74bf6178-dca6-4427-901b-44badacb7eee/2156e343-9b45-4780-9034-2535dd910fa6"
-          (reference "Q1") (unit 1)
-        )
         (path "/74bf6178-dca6-4427-901b-44badacb7eee/7d25a774-c98a-421e-98be-59f63435153d"
           (reference "Q3") (unit 1)
@@
           (reference "#PWR025") (unit 1)
         )
-        (path "/74bf6178-dca6-4427-901b-44badacb7eee/2156e343-9b45-4780-9034-2535dd910fa6"
-          (reference "#PWR05") (unit 1)
-        )
         (path "/74bf6178-dca6-4427-901b-44badacb7eee/7d25a774-c98a-421e-98be-59f63435153d"
           (reference "#PWR023") (unit 1)
@@
         (path "/74bf6178-dca6-4427-901b-44badacb7eee"
           (reference "#PWR022") (unit 1)
-        )
-        (path "/74bf6178-dca6-4427-901b-44badacb7eee/2156e343-9b45-4780-9034-2535dd910fa6"
-          (reference "#PWR05") (unit 1)
         )
         (path "/74bf6178-dca6-4427-901b-44badacb7eee/7d25a774-c98a-421e-98be-59f63435153d"
@@
       (effects (font (size 1.27 1.27)) (justify left) hide)
     )
+    (property "LCSC" "C10487" (at 134.62 59.69 0)
+      (effects (font (size 1.27 1.27)) hide)
+    )
     (pin "1")
     (pin "2")
@@
         (path "/74bf6178-dca6-4427-901b-44badacb7eee"
           (reference "Q4") (unit 1)
-        )
-        (path "/74bf6178-dca6-4427-901b-44badacb7eee/2156e343-9b45-4780-9034-2535dd910fa6"
-          (reference "Q2") (unit 1)
         )
         (path "/74bf6178-dca6-4427-901b-44badacb7eee/7d25a774-c98a-421e-98be-59f63435153d"
@@
       (effects (font (size 1.27 1.27)) (justify right))
     )
-    (property "Footprint" "Capacitor_SMD:C_0402_1005Metric" (at 115.57 73.66 0)
+    (property "Footprint" "Resistor_SMD:R_0402_1005Metric" (at 115.57 73.66 0)
       (effects (font (size 1.27 1.27)) hide)
     )
@@
       (effects (font (size 1.27 1.27)) hide)
     )
+    (property "LCSC" "C25086" (at 115.57 73.66 0)
+      (effects (font (size 1.27 1.27)) hide)
+    )
     (pin "1")
     (pin "2")
@@
           (reference "R3") (unit 1)
         )
-        (path "/74bf6178-dca6-4427-901b-44badacb7eee/2156e343-9b45-4780-9034-2535dd910fa6"
-          (reference "R1") (unit 1)
-        )
-        (path "/74bf6178-dca6-4427-901b-44badacb7eee/7d25a774-c98a-421e-98be-59f63435153d"
+        (path "/74bf6178-dca6-4427-901b-44badacb7eee/7d25a774-c98a-421e-98be-59f63435153d"
